File: components/ecg_ads1292/pcbs/ecg_ads1292/kicad/egc_ads1292.kicad_pcb (KiCad board)
At the start: 2 copper layers, 120 x 52.5 mm, 87 parts, among them IC1 ADS1292, J1 n.p., J2 n.p., J3 n.p., J4 n.p., J5 Conn_02x10_Odd_Even, J6 Conn_02x10_Odd_Even, U1 TPS73033DBVT

Commit message: fix GND via not connected
Routing:
- net GND: vias 72 -> 73
- net (no net): vias 1 -> 0
Changed lines of the file:
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@@
   (via (at 128.5 129) (size 0.8) (drill 0.4) (layers F.Cu B.Cu) (net 2))
   (via (at 128.5 134) (size 0.8) (drill 0.4) (layers F.Cu B.Cu) (net 2))
-  (via (at 123.5 131) (size 0.8) (drill 0.4) (layers F.Cu B.Cu) (net 0))
+  (via (at 123.5 131) (size 0.8) (drill 0.4) (layers F.Cu B.Cu) (net 2))
   (via (at 110 138.5) (size 0.8) (drill 0.4) (layers F.Cu B.Cu) (net 2))
   (via (at 117.5 126) (size 0.8) (drill 0.4) (layers F.Cu B.Cu) (net 2))
