File: components/ecg_ads1292/pcbs/ecg_ads1292/kicad/ecg_ads1292_sensor.sch (KiCad schematic (older format))
At the start: 36 parts, among them IC1 ADS1292, U1 TPS73033DBVT

Commit message: first sim test with ne2 lib, blanks in sheet name removed
Parts:
- C10, C11, C12, C13, C15, C16, C18, C19, C20, C22, C23, C26, C27, C28, C29, C31, C5, C6, C7, C8, C9, IC1, L1, L3, R15, R16, R17, R18, R19, R20, R21, R22, R23, R24, R28, U1: Spice_Netlist_Enabled (none) -> N
Changed lines of the file:
@@
 F 6 "Farnell" H 0   0   50  0001 C CNN "Distributor"
 F 7 "2112849" H 0   0   50  0001 C CNN "Farnell"
+F 8 "N" H 4900 1050 50  0001 C CNN "Spice_Netlist_Enabled"
 	1    4900 1050
 	1    0    0    -1
@@
 F 6 "Farnell" H 0   0   50  0001 C CNN "Distributor"
 F 7 "1907318" H 0   0   50  0001 C CNN "Farnell"
+F 8 "N" H 5850 1050 50  0001 C CNN "Spice_Netlist_Enabled"
 	1    5850 1050
 	1    0    0    -1
@@
 F 6 "Farnell" H 0   0   50  0001 C CNN "Distributor"
 F 7 "1907318" H 0   0   50  0001 C CNN "Farnell"
+F 8 "N" H 6700 1050 50  0001 C CNN "Spice_Netlist_Enabled"
 	1    6700 1050
 	1    0    0    -1
@@
 F 6 "Farnell" H 0   0   50  0001 C CNN "Distributor"
 F 7 "2112849" H 0   0   50  0001 C CNN "Farnell"
+F 8 "N" H 7300 1050 50  0001 C CNN "Spice_Netlist_Enabled"
 	1    7300 1050
 	1    0    0    -1
@@
 F 6 "Farnell" H 0   0   50  0001 C CNN "Distributor"
 F 7 "2611918" H 0   0   50  0001 C CNN "Farnell"
+F 8 "N" H 4400 3000 50  0001 C CNN "Spice_Netlist_Enabled"
 	1    4400 3000
 	0    -1   1    0
@@
 F 6 "Farnell" H 0   0   50  0001 C CNN "Distributor"
 F 7 "2611918" H 0   0   50  0001 C CNN "Farnell"
+F 8 "N" H 4400 3300 50  0001 C CNN "Spice_Netlist_Enabled"
 	1    4400 3300
 	0    -1   1    0
@@
 F 6 "Farnell" H 0   0   50  0001 C CNN "Distributor"
 F 7 "2494294" H 0   0   50  0001 C CNN "Farnell"
+F 8 "N" H 5850 5300 50  0001 C CNN "Spice_Netlist_Enabled"
 	1    5850 5300
 	0    1    1    0
@@
 F 6 "Farnell" H 0   0   50  0001 C CNN "Distributor"
 F 7 "1889276" H 0   0   50  0001 C CNN "Farnell"
+F 8 "N" H 5850 5650 50  0001 C CNN "Spice_Netlist_Enabled"
 	1    5850 5650
 	0    1    1    0
@@
 F 6 "Farnell" H 0   0   50  0001 C CNN "Distributor"
 F 7 "2112849" H 0   0   50  0001 C CNN "Farnell"
+F 8 "N" H 5400 5300 50  0001 C CNN "Spice_Netlist_Enabled"
 	1    5400 5300
 	-1   0    0    -1
@@
 F 6 "Farnell" H 0   0   50  0001 C CNN "Distributor"
 F 7 "2112849" H 0   0   50  0001 C CNN "Farnell"
+F 8 "N" H 5100 5300 50  0001 C CNN "Spice_Netlist_Enabled"
 	1    5100 5300
 	-1   0    0    -1
@@
 F 5 "Farnell" H 0   0   50  0001 C CNN "Distributor"
 F 6 "1738916" H 0   0   50  0001 C CNN "Farnell"
+F 7 "N" H 5800 1850 50  0001 C CNN "Spice_Netlist_Enabled"
 	1    5800 1850
 	1    0    0    -1
@@
 F 5 "Farnell" H 0   0   50  0001 C CNN "Distributor"
 F 6 "1692517" H 0   0   50  0001 C CNN "Farnell"
+F 7 "N" H 5500 1850 50  0001 C CNN "Spice_Netlist_Enabled"
 	1    5500 1850
 	1    0    0    -1
@@
 F 5 "C0G/NPO" H 0   0   50  0001 C CNN "Comment"
 F 6 "" H 0   0   50  0001 C CNN "Farnell"
+F 7 "N" H 4900 1850 50  0001 C CNN "Spice_Netlist_Enabled"
 	1    4900 1850
 	1    0    0    -1
@@
 F 5 "Farnell" H 0   0   50  0001 C CNN "Distributor"
 F 6 "1739145" H 0   0   50  0001 C CNN "Farnell"
+F 7 "N" H 7450 3600 50  0001 C CNN "Spice_Netlist_Enabled"
 	1    7450 3600
 	0    1    1    0
@@
 F 5 "Farnell" H 0   0   50  0001 C CNN "Distributor"
 F 6 "1739145" H 0   0   50  0001 C CNN "Farnell"
+F 7 "N" H 7450 3000 50  0001 C CNN "Spice_Netlist_Enabled"
 	1    7450 3000
 	0    1    1    0
@@
 F 5 "Farnell" H 0   0   50  0001 C CNN "Distributor"
 F 6 "1669719" H 0   0   50  0001 C CNN "Farnell"
+F 7 "N" H 5400 850 50  0001 C CNN "Spice_Netlist_Enabled"
 	1    5400 850
 	0    -1   -1   0
@@
 F 5 "Farnell" H -600 -950 50  0001 C CNN "Distributor"
 F 6 "1469825" H -600 -950 50  0001 C CNN "Farnell"
+F 7 "N" H 1200 3250 50  0001 C CNN "Spice_Netlist_Enabled"
 	1    1200 3250
 	0    -1   -1   0
@@
 F 6 "Farnell" H -800 -950 50  0001 C CNN "Distributor"
 F 7 "1865491" H -800 -950 50  0001 C CNN "Farnell"
+F 8 "N" H 1450 3550 50  0001 C CNN "Spice_Netlist_Enabled"
 	1    1450 3550
 	1    0    0    -1
@@
 F 5 "Farnell" H 1850 2350 50  0001 C CNN "Distributor"
 F 6 "1738916" H 1850 2350 50  0001 C CNN "Farnell"
+F 7 "N" H 7650 4200 50  0001 C CNN "Spice_Netlist_Enabled"
 	1    7650 4200
 	0    -1   -1   0
@@
 F 5 "Farnell" H 1850 2450 50  0001 C CNN "Distributor"
 F 6 "1738916" H 1850 2450 50  0001 C CNN "Farnell"
+F 7 "N" H 7650 4300 50  0001 C CNN "Spice_Netlist_Enabled"
 	1    7650 4300
 	0    1    1    0
@@
 F 5 "Farnell" H -1600 800 50  0001 C CNN "Distributor"
 F 6 "1135395" H -1600 800 50  0001 C CNN "Farnell"
+F 7 "N" H 2850 6650 50  0001 C CNN "Spice_Netlist_Enabled"
 	1    2850 6650
 	1    0    0    -1
@@
 F 5 "Farnell" H -1600 800 50  0001 C CNN "Distributor"
 F 6 "1907318" H -1600 800 50  0001 C CNN "Farnell"
+F 7 "N" H 1900 7000 50  0001 C CNN "Spice_Netlist_Enabled"
 	1    1900 7000
 	1    0    0    -1
@@
 F 5 "Farnell" H -1600 800 50  0001 C CNN "Distributor"
 F 6 "2496825" H -1600 800 50  0001 C CNN "Farnell"
+F 7 "N" H 3400 7000 50  0001 C CNN "Spice_Netlist_Enabled"
 	1    3400 7000
 	1    0    0    -1
@@
 F 5 "Farnell" H -1000 800 50  0001 C CNN "Distributor"
 F 6 "1669719" H -1000 800 50  0001 C CNN "Farnell"
+F 7 "N" H 1400 6550 50  0001 C CNN "Spice_Netlist_Enabled"
 	1    1400 6550
 	0    1    1    0
@@
 F 5 "Farnell" H -1600 800 50  0001 C CNN "Distributor"
 F 6 "1797012" H -1600 800 50  0001 C CNN "Farnell"
+F 7 "N" H 1600 7000 50  0001 C CNN "Spice_Netlist_Enabled"
 	1    1600 7000
 	1    0    0    -1
@@
 F 3 "" H 5200 3250 60  0001 C CNN
 F 4 "Lukas Holzapfel" H 5750 3650 60  0001 C CNN "Created"
+F 5 "N" H 5900 3800 50  0001 C CNN "Spice_Netlist_Enabled"
 	1    5900 3800
 	1    0    0    -1
@@
 F 5 "Farnell" H -600 -100 50  0001 C CNN "Distributor"
 F 6 "1469825" H -600 -100 50  0001 C CNN "Farnell"
+F 7 "N" H 1200 4100 50  0001 C CNN "Spice_Netlist_Enabled"
 	1    1200 4100
 	0    -1   -1   0
@@
 F 6 "Farnell" H -800 -100 50  0001 C CNN "Distributor"
 F 7 "1865491" H -800 -100 50  0001 C CNN "Farnell"
+F 8 "N" H 1450 4400 50  0001 C CNN "Spice_Netlist_Enabled"
 	1    1450 4400
 	1    0    0    -1
@@
 F 5 "Farnell" H -600 750 50  0001 C CNN "Distributor"
 F 6 "1469825" H -600 750 50  0001 C CNN "Farnell"
+F 7 "N" H 1200 4950 50  0001 C CNN "Spice_Netlist_Enabled"
 	1    1200 4950
 	0    -1   -1   0
@@
 F 6 "Farnell" H -800 750 50  0001 C CNN "Distributor"
 F 7 "1865491" H -800 750 50  0001 C CNN "Farnell"
+F 8 "N" H 1450 5250 50  0001 C CNN "Spice_Netlist_Enabled"
 	1    1450 5250
 	1    0    0    -1
@@
 F 6 "Farnell" H -300 -800 50  0001 C CNN "Distributor"
 F 7 "1865491" H -300 -800 50  0001 C CNN "Farnell"
+F 8 "N" H 1950 3700 50  0001 C CNN "Spice_Netlist_Enabled"
 	1    1950 3700
 	1    0    0    -1
@@
 F 6 "Farnell" H -300 0   50  0001 C CNN "Distributor"
 F 7 "1865491" H -300 0   50  0001 C CNN "Farnell"
+F 8 "N" H 1950 4500 50  0001 C CNN "Spice_Netlist_Enabled"
 	1    1950 4500
 	1    0    0    -1
@@
 F 5 "C0G/NPO" H 450 350 50  0001 C CNN "Comment"
 F 6 "" H 450 350 50  0001 C CNN "Farnell"
+F 7 "N" H 5350 2200 50  0001 C CNN "Spice_Netlist_Enabled"
 	1    5350 2200
 	0    1    1    0
@@
 F 5 "Farnell" H 0   0   50  0001 C CNN "Distributor"
 F 6 "1469746" H 0   0   50  0001 C CNN "Farnell"
+F 7 "N" H 5200 1850 50  0001 C CNN "Spice_Netlist_Enabled"
 	1    5200 1850
 	1    0    0    -1
@@
 F 5 "Farnell" H -1600 800 50  0001 C CNN "Distributor"
 F 6 "1797012" H -1600 800 50  0001 C CNN "Farnell"
+F 7 "N" H 3800 7000 50  0001 C CNN "Spice_Netlist_Enabled"
 	1    3800 7000
 	1    0    0    -1
@@
 F 5 "Farnell" H 0   300 50  0001 C CNN "Distributor"
 F 6 "1739145" H 0   300 50  0001 C CNN "Farnell"
+F 7 "N" H 7450 3900 50  0001 C CNN "Spice_Netlist_Enabled"
 	1    7450 3900
 	0    1    1    0
