File: components/ecg_ads1292/pcbs/ecg_ads1292_main/kicad/ecg_ads1292_main.sch (KiCad schematic (older format))
At the start: 13 parts, among them J1 Conn_02x04_Odd_Even, P1 Conn_02x20_Odd_Even

Commit message: schematic passes erc with two accpted warnings
Connections:
- no-connect marks 0 -> 21
Other:
- moved on the sheet: J1, R1, R2, R3, TP15
