File: components/ecg_ads1292/pcbs/ecg_ads1292_main/kicad/ecg_ads1292_main.kicad_pcb (KiCad board)
At the start: 2 copper layers, 65 x 36 mm, 52 parts, among them IC1 ADS1292, J1 Conn_02x04_Odd_Even, P1 Conn_02x20_Odd_Even, U1 TPS73033DBVT

Commit message: ecg_ads1292: update part fields
Parts:
- C1, C2, C3: value 47p C0G 50V -> 47p 50V
- C13: value 470p -> 470p 50V
- IC1: value ADS1292 -> ADS1292IPBSR
- MK1, MK2, MK3, MK4: value M2.5 -> n.p.
- TP15, TP5: value (none) -> n.p.
Changed lines of the file:
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@@
       (effects (font (size 1 1) (thickness 0.15)))
     )
-    (fp_text value " " (at 0 -2.8) (layer F.Fab)
+    (fp_text value n.p. (at 0 -2.8) (layer F.Fab)
       (effects (font (size 1 1) (thickness 0.15)))
     )
@@
       (effects (font (size 1 1) (thickness 0.15)))
     )
-    (fp_text value " " (at 0 -2.8) (layer F.Fab)
+    (fp_text value n.p. (at 0 -2.8) (layer F.Fab)
       (effects (font (size 1 1) (thickness 0.15)))
     )
@@
       (effects (font (size 1 1) (thickness 0.15)))
     )
-    (fp_text value ADS1292 (at 0 4.88 90) (layer F.Fab)
+    (fp_text value ADS1292IPBSR (at 0 4.88 90) (layer F.Fab)
       (effects (font (size 1 1) (thickness 0.15)))
     )
@@
       (effects (font (size 1 1) (thickness 0.15)))
     )
-    (fp_text value 470p (at 0 1.43) (layer F.Fab)
+    (fp_text value "470p 50V" (at 0 1.43) (layer F.Fab)
       (effects (font (size 1 1) (thickness 0.15)))
     )
@@
       (effects (font (size 1 1) (thickness 0.15)))
     )
-    (fp_text value "47p C0G 50V" (at 0 1.43 90) (layer F.Fab)
+    (fp_text value "47p 50V" (at 0 1.43 90) (layer F.Fab)
       (effects (font (size 1 1) (thickness 0.15)))
     )
@@
       (effects (font (size 1 1) (thickness 0.15)))
     )
-    (fp_text value "47p C0G 50V" (at 0 1.43 90) (layer F.Fab)
+    (fp_text value "47p 50V" (at 0 1.43 90) (layer F.Fab)
       (effects (font (size 1 1) (thickness 0.15)))
     )
@@
       (effects (font (size 1 1) (thickness 0.15)))
     )
-    (fp_text value "47p C0G 50V" (at 0 1.43 90) (layer F.Fab)
+    (fp_text value "47p 50V" (at 0 1.43 90) (layer F.Fab)
       (effects (font (size 1 1) (thickness 0.15)))
     )
@@
       (effects (font (size 1 1) (thickness 0.15)))
     )
-    (fp_text value M2.5 (at 0 3.7) (layer F.Fab)
+    (fp_text value n.p. (at 0 3.7) (layer F.Fab)
       (effects (font (size 1 1) (thickness 0.15)))
     )
@@
       (effects (font (size 1 1) (thickness 0.15)))
     )
-    (fp_text value M2.5 (at 0 3.7) (layer F.Fab)
+    (fp_text value n.p. (at 0 3.7) (layer F.Fab)
       (effects (font (size 1 1) (thickness 0.15)))
     )
@@
       (effects (font (size 1 1) (thickness 0.15)))
     )
-    (fp_text value M2.5 (at 0 3.7 180) (layer F.Fab)
+    (fp_text value n.p. (at 0 3.7 180) (layer F.Fab)
       (effects (font (size 1 1) (thickness 0.15)))
     )
@@
       (effects (font (size 1 1) (thickness 0.15)))
     )
-    (fp_text value M2.5 (at 0 3.7 180) (layer F.Fab)
-      (effects (font (size 1 1) (thickness 0.15)))
-    )
+    (fp_text value n.p. (at 0 3.7 180) (layer F.Fab)
+      (effects (font (size 1 1) (thickness 0.15)))
+    )

Commit message: update parts in pcb
Parts:
- C1, C2, C3: value 47p 50V -> 3n 50V
- C15: value 470p -> 470p 50V
- L1: value MMZ2012R102A -> MMZ2012R102AT000
- R20, R5: value 100 -> n.p.
Changed lines of the file:
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@@
       (effects (font (size 1 1) (thickness 0.15)))
     )
-    (fp_text value 100 (at 0 1.43 90) (layer F.Fab)
+    (fp_text value n.p. (at 0 1.43 90) (layer F.Fab)
       (effects (font (size 1 1) (thickness 0.15)))
     )
@@
       (effects (font (size 1 1) (thickness 0.15)))
     )
-    (fp_text value 100 (at 0 1.43 90) (layer F.Fab)
+    (fp_text value n.p. (at 0 1.43 90) (layer F.Fab)
       (effects (font (size 1 1) (thickness 0.15)))
     )
@@
       (effects (font (size 1 1) (thickness 0.15)))
     )
-    (fp_text value MMZ2012R102A (at 0 1.65 90) (layer F.Fab)
+    (fp_text value MMZ2012R102AT000 (at 0 1.65 90) (layer F.Fab)
       (effects (font (size 1 1) (thickness 0.15)))
     )
@@
       (effects (font (size 1 1) (thickness 0.15)))
     )
-    (fp_text value 470p (at 0 1.43 90) (layer F.Fab)
+    (fp_text value "470p 50V" (at 0 1.43 90) (layer F.Fab)
       (effects (font (size 1 1) (thickness 0.15)))
     )
@@
       (effects (font (size 1 1) (thickness 0.15)))
     )
-    (fp_text value "47p 50V" (at 0 1.43 90) (layer F.Fab)
+    (fp_text value "3n 50V" (at 0 1.43 90) (layer F.Fab)
       (effects (font (size 1 1) (thickness 0.15)))
     )
@@
       (effects (font (size 1 1) (thickness 0.15)))
     )
-    (fp_text value "47p 50V" (at 0 1.43 90) (layer F.Fab)
+    (fp_text value "3n 50V" (at 0 1.43 90) (layer F.Fab)
       (effects (font (size 1 1) (thickness 0.15)))
     )
@@
       (effects (font (size 1 1) (thickness 0.15)))
     )
-    (fp_text value "47p 50V" (at 0 1.43 90) (layer F.Fab)
-      (effects (font (size 1 1) (thickness 0.15)))
-    )
+    (fp_text value "3n 50V" (at 0 1.43 90) (layer F.Fab)
+      (effects (font (size 1 1) (thickness 0.15)))
+    )
