File: resources/template_pcb/kicad/COMPONENT_VARIANT_PCBNAME.sch (KiCad schematic (older format))
At the start: 5 parts, among them P1 Conn_02x20_Odd_Even

Commit message: update check lists
Parts:
- added MK5, MK6: M2.5, MountingHole:MountingHole_2.7mm_M2.5, symbol Mechanical:MountingHole
Connections:
- net labels added: +3.3VA, +5VA, +5VD, SENS_3V3_ANA, SENS_5V_ANA, SENS_5V_DIG, SENS_GPIO0, SENS_GPIO1, SENS_INT_BPM, SENS_INT_ECG, SENS_INT_SPO2, SENS_MISO, SENS_MOSI, SENS_SCL, SENS_SCLK, SENS_SDA, SENS_START, ~SENS_CS_BPM, ~SENS_CS_ECG, ~SENS_CS_SPO2, ~SENS_RST_BPM, ~SENS_RST_ECG, ~SENS_RST_SPO2
- net labels removed: +5V, GPIO10(SPI0_MOSI), GPIO11(SPI0_SCK), GPIO14(TXD0), GPIO15(RXD0), GPIO17(GEN0), GPIO18(GEN1)(PWM0), GPIO2(SDA1), GPIO22(GEN3), GPIO23(GEN4), GPIO24(GEN5), GPIO25(GEN6), GPIO27(GEN2), GPIO3(SCL1), GPIO4(GCLK), GPIO7(SPI1_CE_N), GPIO8(SPI0_CE_N), GPIO9(SPI0_MISO)
Other:
- note added: "ATTENTION: max. 300mA for both 5V rails together allowed on RPi."
- note added: "ATTENTION: max. 30mA for both 3.3V rails together allowed on RPi."
- note added: "Interconnect"
- note added: "Mounting"
- note added: "Pins 1 to 26 belong to the sensor bus.\nPins 27 to 40 are named according to RPi header pin names."
- moved on the sheet: MK1, MK2, MK3, MK4, P1

Commit message: add chip select mux in pcb template
Parts:
- added R1, R2, R3: n.p., Resistor_SMD:R_0603_1608Metric_Pad1.05x0.95mm_HandSolder, symbol Device:R_Small
Connections:
- net labels added: ~CS
- wire segments 52 -> 58
Changed lines of the file:
@@
 	14150 4250 15200 4250
 Wire Wire Line
-	14150 3650 15200 3650
-Wire Wire Line
 	14150 3750 15200 3750
 Wire Wire Line
-	14150 3450 15200 3450
-Wire Wire Line
-	14150 3550 15200 3550
+	14150 3450 15350 3450
+Wire Wire Line
+	14150 3550 15350 3550
 Wire Wire Line
 	14150 3150 15200 3150
@@
 	1    0    0    -1
 $EndComp
+$Comp
+L Device:R_Small R1
+U 1 1 5EA7E07E
+P 15450 3450
+F 0 "R1" V 15400 3300 50  0000 C CNN
+F 1 "n.p." V 15400 3600 50  0000 C CNN
+F 2 "Resistor_SMD:R_0603_1608Metric_Pad1.05x0.95mm_HandSolder" H 15450 3450 50  0001 C CNN
+F 3 "~" H 15450 3450 50  0001 C CNN
+	1    15450 3450
+	0    1    1    0
+$EndComp
+Wire Wire Line
+	14150 3650 15350 3650
+Wire Wire Line
+	15550 3650 15700 3650
+Wire Wire Line
+	15700 3650 15700 3550
+Wire Wire Line
+	15550 3450 15700 3450
+Connection ~ 15700 3450
+Wire Wire Line
+	15700 3450 16000 3450
+Wire Wire Line
+	15550 3550 15700 3550
+Connection ~ 15700 3550
+Wire Wire Line
+	15700 3550 15700 3450
+Text Label 16000 3450 2    50   ~ 0
+~CS
+$Comp
+L Device:R_Small R2
+U 1 1 5EA881A8
+P 15450 3550
+F 0 "R2" V 15400 3400 50  0000 C CNN
+F 1 "n.p." V 15400 3700 50  0000 C CNN
+F 2 "Resistor_SMD:R_0603_1608Metric_Pad1.05x0.95mm_HandSolder" H 15450 3550 50  0001 C CNN
+F 3 "~" H 15450 3550 50  0001 C CNN
+	1    15450 3550
+	0    1    1    0
+$EndComp
+$Comp
+L Device:R_Small R3
+U 1 1 5EA8833D
+P 15450 3650
+F 0 "R3" V 15400 3500 50  0000 C CNN
+F 1 "n.p." V 15400 3800 50  0000 C CNN
+F 2 "Resistor_SMD:R_0603_1608Metric_Pad1.05x0.95mm_HandSolder" H 15450 3650 50  0001 C CNN
+F 3 "~" H 15450 3650 50  0001 C CNN
+	1    15450 3650
+	0    1    1    0
+$EndComp
 $EndSCHEMATC
