File: resources/templates/template_pcb/kicad/COMPONENT_VARIANT_PCBNAME.kicad_pcb (KiCad board)
At the start: 2 copper layers, 65 x 56 mm, 10 parts, among them P1 Conn_02x20_Odd_Even

Commit message: improve pcb template
Other:
- net class Default: trace_width 0.2 -> 0.25
- rule trace_min: 0.1524 -> 0.25
- board text added: "ATTENTION: P1 SHOULD BE INSERTED FROM THE BOTTOM OF THE BOARD"
- board text added: "All connectors (except for P1) must be angled and must be placed on this edge pointing downwards."
- board text added: "Cadus e.V. lifesensor COMPONENT_VARIANT_PCBNAME Rev. 0"
- board text added: "RASPBERRY-PI 40-PIN ADDON BOARD VIEW FROM TOP NOTE: P1 SHOULD BE INSERTED FROM THE BOTTOM OF THE BOARD NOTE: remove pcb edge below MK3/MK4 or MK5/MK6 depending on the board size you need."
- board text added: "place all connectors here"
- board text removed: "All connectors except the 40 pin header must be angled and must be placed on this edge pointing downwards."
- board text removed: "RASPBERRY-PI 40-PIN ADDON BOARD VIEW FROM TOP NOTE: P1 SHOULD BE FITTED ON THE REVERSE OF THE BOARD NOTE: remove pcb edge below MK3/MK4 or MK5/MK6 depending on the board size you need."
Changed lines of the file:
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@@
   (general
     (thickness 1.6)
-    (drawings 13)
+    (drawings 21)
     (tracks 32)
     (zones 0)
@@
     (zone_clearance 0.508)
     (zone_45_only no)
-    (trace_min 0.1524)
+    (trace_min 0.25)
     (via_size 0.9)
     (via_drill 0.5)
@@
   (net_class Default "This is the default net class."
     (clearance 0.2)
-    (trace_width 0.2)
+    (trace_width 0.25)
     (via_dia 0.9)
     (via_drill 0.5)
     (uvia_dia 0.5)
     (uvia_drill 0.1)
-    (add_net +3.3VA)
-    (add_net +3V3)
-    (add_net +5VA)
-    (add_net +5VD)
+    (diff_pair_width 0.25)
+    (diff_pair_gap 0.25)
     (add_net "/GPIO12(PWM0)")
     (add_net "/GPIO13(PWM1)")
@@
     (add_net /~SENS_RST_ECG)
     (add_net /~SENS_RST_SPO2)
-    (add_net GND)
   )
   (net_class Power ""
@@
     (uvia_dia 0.5)
     (uvia_drill 0.1)
+    (diff_pair_width 0.25)
+    (diff_pair_gap 0.25)
+    (add_net +3.3VA)
+    (add_net +3V3)
+    (add_net +5VA)
+    (add_net +5VD)
+    (add_net GND)
   )
   (module Resistor_SMD:R_0603_1608Metric_Pad1.05x0.95mm_HandSolder (layer F.Cu)
@@
     (pad 1 np_thru_hole circle (at 0 0 180) (size 2.7 2.7) (drill 2.7) (layers *.Cu *.Mask))
   )
-  (gr_text "All connectors except the 40 pin header must be angled\nand must be placed on this edge pointing downwards." (at 200 158) (layer Dwgs.User)
+  (gr_text "ATTENTION: P1 SHOULD BE INSERTED FROM THE BOTTOM OF THE BOARD" (at 232.5 93) (layer F.SilkS)
+    (effects (font (size 1.5 1.25) (thickness 0.25)))
+  )
+  (gr_text "place all connectors here" (at 232 145) (layer Dwgs.User)
+    (effects (font (size 3 2) (thickness 0.3)))
+  )
+  (gr_text "Cadus e.V. lifesensor\nCOMPONENT_VARIANT_PCBNAME\nRev. 0" (at 207.5 103 270) (layer F.Mask)
+    (effects (font (size 1.5 1.25) (thickness 0.3)) (justify left))
+  )
+  (gr_text "Cadus e.V. lifesensor\nCOMPONENT_VARIANT_PCBNAME\nRev. 0" (at 207.5 103 270) (layer F.Cu)
+    (effects (font (size 1.5 1.25) (thickness 0.3)) (justify left))
+  )
+  (gr_line (start 257 140) (end 208 140) (layer Dwgs.User) (width 0.12))
+  (gr_line (start 257 150) (end 257 140) (layer Dwgs.User) (width 0.12))
+  (gr_line (start 208 150) (end 257 150) (layer Dwgs.User) (width 0.12))
+  (gr_line (start 208 140) (end 208 150) (layer Dwgs.User) (width 0.12))
+  (gr_text "All connectors (except for P1) must be angled\nand must be placed on this edge pointing downwards." (at 200 158) (layer Dwgs.User)
     (effects (font (size 2 1.7) (thickness 0.12)) (justify left))
   )
@@
   (gr_line (start 203 150) (end 262 150) (layer Edge.Cuts) (width 0.1))
   (gr_line (start 200 97) (end 200 147) (layer Edge.Cuts) (width 0.1))
-  (gr_text "RASPBERRY-PI 40-PIN ADDON BOARD\nVIEW FROM TOP\nNOTE: P1 SHOULD BE FITTED ON THE REVERSE OF THE BOARD\nNOTE: remove pcb edge below MK3/MK4 or MK5/MK6 depending on the board size you need." (at 200 83) (layer Dwgs.User)
+  (gr_text "RASPBERRY-PI 40-PIN ADDON BOARD\nVIEW FROM TOP\nNOTE: P1 SHOULD BE INSERTED FROM THE BOTTOM OF THE BOARD\nNOTE: remove pcb edge below MK3/MK4 or MK5/MK6 depending on the board size you need." (at 200 83) (layer Dwgs.User)
     (effects (font (size 2 1.7) (thickness 0.12)) (justify left))
   )
